Commit message: Add dataset and 3d point generation of pcd

File: elfin-robot/elfin_description/urdf/S20_with_gripper_38cm.urdf (robot description, URDF)
Before this commit: robot S20, 15 links, 14 joints
Joints:
- joint ee_link_joint: origin xyz=-0.155 -0.0315 0 rpy=-1.5707 0 0 -> xyz=0.035 -0.155 0 rpy=-1.5707 0 1.5707

File: elfin-robot/elfin_description/urdf/S20_with_gripper_48cm.urdf (robot description, URDF)
Before this commit: robot S20, 16 links, 15 joints
Joints:
- joint ee_link_joint: origin xyz=-0.155 -0.0315 0 rpy=-1.5707 0 0 -> xyz=0.035 -0.155 0 rpy=-1.5707 0 1.5707

File: elfin-robot/elfin_description/urdf/S20_with_gripper_58cm.urdf (robot description, URDF)
Before this commit: robot S20, 17 links, 16 joints
Joints:
- joint ee_link_joint: origin xyz=-0.155 -0.0315 0 rpy=-1.5707 0 0 -> xyz=0.035 -0.155 0 rpy=-1.5707 0 1.5707

File: elfin-robot/elfin_description/urdf/S20_with_gripper_68cm.urdf (robot description, URDF)
Before this commit: robot S20, 18 links, 17 joints
Joints:
- joint ee_link_joint: origin xyz=-0.155 -0.0315 0 rpy=-1.5707 0 0 -> xyz=0.035 -0.155 0 rpy=-1.5707 0 1.5707
