Commit message: Add base for S20 48cm

File: elfin-robot/elfin_description/urdf/S20_with_gripper_48cm.urdf (robot description, URDF)
Before this commit: robot S20, 16 links, 15 joints
Links:
- removed link world
- added link world_base0; visual box size=0.1 0.1 0.1
- added link world_base1; visual box size=0.1 0.1 0.1
- added link world_base2; visual box size=0.3 0.3 1.3
Joints:
- removed joint world_base
- added joint world_base0: type prismatic, parent world_base0, child world_base1, origin xyz=0 0 0 rpy=0 0 0, axis 1 0 0, limit lower=-5 upper=5
- added joint world_base1: type prismatic, parent world_base1, child world_base2, origin xyz=0 0 0 rpy=0 0 0, axis 0 1 0, limit lower=-5 upper=5
- added joint world_base2: type fixed, parent world_base2, child elfin_base_link, origin xyz=0 0 1.3 rpy=0 0 0
